File: electronics/v1/sandsim.sch (KiCad schematic (older format))
At the start: 14 parts, among them SW1 SW_SPST, U1 SeeeduinoXIAO, U2 EA-DOGM128W-6, U3 MPU_Breakout

Commit message: update for publishing on hackaday
Parts:
- U1: symbol XIAO:SeeeduinoXIAO -> sandsim-rescue:SeeeduinoXIAO-XIAO
- U2: symbol DOGM128:EA-DOGM128W-6 -> sandsim-rescue:EA-DOGM128W-6-DOGM128
Changed lines of the file:
@@
 $EndComp
 $Comp
-L XIAO:SeeeduinoXIAO U1
+L sandsim-rescue:SeeeduinoXIAO-XIAO U1
 U 1 1 62D227C0
 P 2800 2700
@@
 	4250 5450 4500 5450
 $Comp
-L DOGM128:EA-DOGM128W-6 U2
+L sandsim-rescue:EA-DOGM128W-6-DOGM128 U2
 U 1 1 62D27F39
 P 5650 2650
@@
 $EndComp
 $Comp
-L DOGM128:EA-DOGM128W-6 U2
+L sandsim-rescue:EA-DOGM128W-6-DOGM128 U2
 U 2 1 62D28F12
 P 6300 5300
